File: hw/relelauta/v2/relelauta/relelauta.sch (KiCad schematic (older format))
At the start: 100 parts, among them J1 stack[0..3], J2 stack[0..3], J3 stack[0..3], J4 stack[0..3], Q1 IRLZ44N, Q10 IRLZ44N, Q11 IRLZ44N, Q12 IRLZ44N, Q13 IRLZ44N, Q14 IRLZ44N, Q15 IRLZ44N, Q16 IRLZ44N, Q2 IRLZ44N, Q3 IRLZ44N, Q4 IRLZ44N, Q5 IRLZ44N, Q6 IRLZ44N, Q7 IRLZ44N, Q8 IRLZ44N, Q9 IRLZ44N

Commit message: Finish laying out relelauta v2.0 PCB. Minor tweaks to motherboard.
Parts:
- added C33, C34: 1u, Capacitor_SMD:C_0603_1608Metric, symbol Device:C_Small
- added D65: LED_12V, LED_SMD:LED_0805_2012Metric, symbol Device:LED_Small
- added D66: LED_5V, LED_SMD:LED_0805_2012Metric, symbol Device:LED_Small
- added D67: LED (sensor power), LED_SMD:LED_0805_2012Metric, symbol Device:LED_Small
- added J10: PSU_Conn, Connector_Molex:Molex_Mini-Fit_Jr_5566-06A_2x03_P4.20mm_Vertical, symbol Connector_Generic:Conn_02x03_Counter_Clockwise
- added J11, J12, J13, J14, J15, J16, J17, J18, J19, J20, J21, J22, J23, J24, J25, J7: Conn_sensor, Connector_PinHeader_2.54mm:PinHeader_1x03_P2.54mm_Horizontal, symbol Connector:Conn_01x03_Male
- added J5: STACK_5V, Connector_PinSocket_2.54mm:PinSocket_1x02_P2.54mm_Vertical, symbol Connector_Generic:Conn_01x02
- added J6: STACK_GND, Connector_PinSocket_2.54mm:PinSocket_1x02_P2.54mm_Vertical, symbol Connector_Generic:Conn_01x02
- added R33, R34, R35: 10k, Resistor_SMD:R_0805_2012Metric, symbol Device:R_Small
- added U1: TLV75533PDBV, Package_TO_SOT_SMD:SOT-23-5, symbol Regulator_Linear:TLV75533PDBV
- renumbered D2 to D1, D11 to D10, D19 to D11, D27 to D12, D5 to D13, D12 to D14, D20 to D15, D28 to D16, D6 to D17, D7 to D18, D8 to D19, D9 to D2, D13 to D20, D14 to D21, D15 to D22, D16 to D23, D21 to D24, D22 to D25, D23 to D26, D24 to D27, D29 to D28, D30 to D29, D17 to D3, D31 to D30, D32 to D31, D1 to D32, D25 to D4, D3 to D5, D10 to D6, D18 to D7, D26 to D8, D4 to D9, L7 to L10, L15 to L12, L4 to L13, L8 to L14, L12 to L15, L5 to L2, L9 to L3, L13 to L4, L2 to L5, L10 to L7, L14 to L8, L3 to L9, Q7 to Q10, Q15 to Q12, Q4 to Q13, Q8 to Q14, Q12 to Q15, Q5 to Q2, Q9 to Q3, Q13 to Q4, Q2 to Q5, Q10 to Q7, Q14 to Q8, Q3 to Q9
Connections:
- net +12V: now also D65.2 (A), J10.1 (Pin_1), J10.3 (Pin_3)
- net GND: now also C33.2, C34.2, J10.4 (Pin_4), J10.6 (Pin_6), J11.1 (Pin_1), J12.1 (Pin_1), J13.1 (Pin_1), J14.1 (Pin_1), J15.1 (Pin_1), J16.1 (Pin_1), J17.1 (Pin_1), J18.1 (Pin_1), J19.1 (Pin_1), J20.1 (Pin_1), J21.1 (Pin_1), J22.1 (Pin_1), J23.1 (Pin_1), J24.1 (Pin_1), J25.1 (Pin_1), J6.1 (Pin_1), J6.2 (Pin_2), J7.1 (Pin_1), R33.2, R34.2, R35.2, U1.2 (GND)
- net s0: now also J7.3 (Pin_3)
- net s1: now also J18.3 (Pin_3)
- net s10: now also J15.3 (Pin_3)
- net s11: now also J23.3 (Pin_3)
- net s12: now also J16.3 (Pin_3)
- net s13: now also J24.3 (Pin_3)
- net s14: now also J17.3 (Pin_3)
- net s15: now also J25.3 (Pin_3)
- net s2: now also J11.3 (Pin_3)
- net s3: now also J19.3 (Pin_3)
- net s4: now also J12.3 (Pin_3)
- net s5: now also J20.3 (Pin_3)
- net s6: now also J13.3 (Pin_3)
- net s7: now also J21.3 (Pin_3)
- net s8: now also J14.3 (Pin_3)
- net s9: now also J22.3 (Pin_3)
- new net: D67.1 (K), R35.1
- new net: D65.1 (K), R33.1
- new net: D66.1 (K), R34.1
- new net +5V: C33.1, D66.2 (A), J10.5 (Pin_5), J5.1 (Pin_1), J5.2 (Pin_2), U1.1 (IN), U1.3 (EN)
- new net 3.3V_sensor: C34.1, D67.2 (A), J11.2 (Pin_2), J12.2 (Pin_2), J13.2 (Pin_2), J14.2 (Pin_2), J15.2 (Pin_2), J16.2 (Pin_2), J17.2 (Pin_2), J18.2 (Pin_2), J19.2 (Pin_2), J20.2 (Pin_2), J21.2 (Pin_2), J22.2 (Pin_2), J23.2 (Pin_2), J24.2 (Pin_2), J25.2 (Pin_2), J7.2 (Pin_2), U1.5 (OUT)
- no-connect marks 0 -> 1
Other:
- note added: "Sensor connectors"
- note added: "each sensor draws around 2mA from 3.3V line\nthere are 16 sensor boards\ncomparator is also powered from 3.3V line\n= 32mA\naround 50mA should be fine\n"
