File: hw/relelauta/v2/relelauta/relelauta.kicad_pcb (KiCad board)
At the start: 2 copper layers, 100 x 100 mm, 150 parts, among them J1 stack[0..3], J10 PSU_Conn, J11 Conn_sensor, J12 Conn_sensor, J13 Conn_sensor, J14 Conn_sensor, J15 Conn_sensor, J16 Conn_sensor, J17 Conn_sensor, J18 Conn_sensor, J19 Conn_sensor, J2 stack[0..3], J20 Conn_sensor, J21 Conn_sensor, J22 Conn_sensor, J23 Conn_sensor, J24 Conn_sensor, J25 Conn_sensor, J3 stack[0..3], J4 stack[0..3], J5 STACK_5V, J6 STACK_GND, J7 Conn_sensor, J8 RGB stack in, Q1 IRLZ44N, Q10 IRLZ44N, Q11 IRLZ44N, Q12 IRLZ44N, Q13 IRLZ44N, Q14 IRLZ44N, Q15 IRLZ44N, Q16 IRLZ44N, Q2 IRLZ44N, Q3 IRLZ44N, Q4 IRLZ44N, Q5 IRLZ44N, Q6 IRLZ44N, Q7 IRLZ44N, Q8 IRLZ44N, Q9 IRLZ44N, U1 TLV75533PDBV

Commit message: Add missing silkscreen markings
Other:
- board text added: "+"
- board text added: "+12V"
- board text added: "+5V"
- board text added: "NC"
Changed lines of the file:
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@@
   (general
     (thickness 1.6)
-    (drawings 41)
+    (drawings 114)
     (tracks 955)
     (zones 0)
@@
     )
   )
+  (gr_text + (at 166.39 89.4) (layer F.SilkS)
+    (effects (font (size 0.8 0.8) (thickness 0.1)))
+  )
+  (gr_text + (at 166.33 85.92) (layer F.SilkS)
+    (effects (font (size 0.8 0.8) (thickness 0.1)))
+  )
+  (gr_text + (at 166.2 82.45) (layer F.SilkS)
+    (effects (font (size 0.8 0.8) (thickness 0.1)))
+  )
+  (gr_text + (at 149.87 138.87) (layer F.SilkS)
+    (effects (font (size 0.8 0.8) (thickness 0.1)))
+  )
+  (gr_text + (at 165.1 135.79) (layer F.SilkS)
+    (effects (font (size 0.8 0.8) (thickness 0.1)))
+  )
+  (gr_text + (at 177.66 127.36) (layer F.SilkS)
+    (effects (font (size 0.8 0.8) (thickness 0.1)))
+  )
+  (gr_text + (at 185.91 114.93) (layer F.SilkS)
+    (effects (font (size 0.8 0.8) (thickness 0.1)))
+  )
+  (gr_text + (at 188.9 100.03) (layer F.SilkS)
+    (effects (font (size 0.8 0.8) (thickness 0.1)))
+  )
+  (gr_text + (at 186.09 85.13) (layer F.SilkS)
+    (effects (font (size 0.8 0.8) (thickness 0.1)))
+  )
+  (gr_text + (at 177.53 72.47) (layer F.SilkS)
+    (effects (font (size 0.8 0.8) (thickness 0.1)))
+  )
+  (gr_text + (at 165.17 64.22) (layer F.SilkS)
+    (effects (font (size 0.8 0.8) (thickness 0.1)))
+  )
+  (gr_text + (at 149.79 61.33) (layer F.SilkS)
+    (effects (font (size 0.8 0.8) (thickness 0.1)))
+  )
+  (gr_text + (at 135.14 64.27) (layer F.SilkS)
+    (effects (font (size 0.8 0.8) (thickness 0.1)))
+  )
+  (gr_text + (at 122.45 72.51) (layer F.SilkS)
+    (effects (font (size 0.8 0.8) (thickness 0.1)))
+  )
+  (gr_text + (at 114.03 85.12) (layer F.SilkS)
+    (effects (font (size 0.8 0.8) (thickness 0.1)))
+  )
+  (gr_text + (at 110.93 100.03) (layer F.SilkS)
+    (effects (font (size 0.8 0.8) (thickness 0.1)))
+  )
+  (gr_text + (at 113.89 114.92) (layer F.SilkS)
+    (effects (font (size 0.8 0.8) (thickness 0.1)))
+  )
+  (gr_text + (at 122.44 127.41) (layer F.SilkS)
+    (effects (font (size 0.8 0.8) (thickness 0.1)))
+  )
+  (gr_text + (at 135.3 135.86) (layer F.SilkS)
+    (effects (font (size 0.8 0.8) (thickness 0.1)))
+  )
+  (gr_text NC (at 149.94 94.62) (layer B.SilkS)
+    (effects (font (size 0.8 0.8) (thickness 0.1)) (justify mirror))
+  )
+  (gr_text +5V (at 150.13 105.48) (layer B.SilkS)
+    (effects (font (size 0.8 0.8) (thickness 0.1)) (justify mirror))
+  )
+  (gr_text GND (at 145.79 105.51) (layer B.SilkS)
+    (effects (font (size 0.8 0.8) (thickness 0.1)) (justify mirror))
+  )
+  (gr_text GND (at 154.29 105.51) (layer B.SilkS)
+    (effects (font (size 0.8 0.8) (thickness 0.1)) (justify mirror))
+  )
+  (gr_text +12V (at 154.26 94.57) (layer B.SilkS)
+    (effects (font (size 0.8 0.8) (thickness 0.1)) (justify mirror))
+  )
+  (gr_text +12V (at 145.79 94.53) (layer B.SilkS)
+    (effects (font (size 0.8 0.8) (thickness 0.1)) (justify mirror))
+  )
+  (gr_text GND (at 156.819174 147.7719 -348.8) (layer F.SilkS)
+    (effects (font (size 1 1) (thickness 0.15)))
+  )
+  (gr_text S (at 162.013683 146.724305 -348.8) (layer F.SilkS)
+    (effects (font (size 1 1) (thickness 0.15)))
+  )
+  (gr_text + (at 159.489025 147.109793 -348.8) (layer F.SilkS)
+    (effects (font (size 1.5 1.5) (thickness 0.18)))
+  )
+  (gr_text GND (at 174.694938 141.417121 -326.3) (layer F.SilkS)
+    (effects (font (size 1 1) (thickness 0.15)))
+  )
+  (gr_text S (at 179.093141 138.461417 -326.3) (layer F.SilkS)
+    (effects (font (size 1 1) (thickness 0.15)))
+  )
+  (gr_text + (at 176.908181 139.783706 -326.3) (layer F.SilkS)
+    (effects (font (size 1.5 1.5) (thickness 0.18)))
+  )
+  (gr_text + (at 189.974541 126.544098 -303.8) (layer F.SilkS)
+    (effects (font (size 1.5 1.5) (thickness 0.18)))
+  )
+  (gr_text S (at 191.487163 124.486314 -303.8) (layer F.SilkS)
+    (effects (font (size 1 1) (thickness 0.15)))
+  )
+  (gr_text GND (at 188.554852 128.900148 -303.8) (layer F.SilkS)
+    (effects (font (size 1 1) (thickness 0.15)))
+  )
+  (gr_text S (at 197.642154 107.009178 -281.3) (layer F.SilkS)
+    (effects (font (size 1 1) (thickness 0.15)))
+  )
+  (gr_text GND (at 196.622153 112.209176 -281.3) (layer F.SilkS)
+    (effects (font (size 1 1) (thickness 0.15)))
+  )
+  (gr_text + (at 197.032153 109.489178 -281.3) (layer F.SilkS)
+    (effects (font (size 1.5 1.5) (thickness 0.18)))
+  )
+  (gr_text S (at 196.796457 88.045492 -258.8) (layer F.SilkS)
+    (effects (font (size 1 1) (thickness 0.15)))
+  )
+  (gr_text GND (at 197.844052 93.240001 -258.8) (layer F.SilkS)
+    (effects (font (size 1 1) (thickness 0.15)))
+  )
+  (gr_text + (at 197.181945 90.57015 -258.8) (layer F.SilkS)
+    (effects (font (size 1.5 1.5) (thickness 0.18)))
+  )
+  (gr_text S (at 188.57357 71.066034 -236.3) (layer F.SilkS)
+    (effects (font (size 1 1) (thickness 0.15)))
+  )
+  (gr_text GND (at 191.529274 75.464237 -236.3) (layer F.SilkS)
+    (effects (font (size 1 1) (thickness 0.15)))
+  )
+  (gr_text + (at 189.895859 73.250994 -236.3) (layer F.SilkS)
+    (effects (font (size 1.5 1.5) (thickness 0.18)))
+  )
+  (gr_text S (at 174.488468 58.342012 -213.8) (layer F.SilkS)
+    (effects (font (size 1 1) (thickness 0.15)))
+  )
+  (gr_text GND (at 178.902302 61.274323 -213.8) (layer F.SilkS)
+    (effects (font (size 1 1) (thickness 0.15)))
+  )
+  (gr_text + (at 176.546251 59.854634 -213.8) (layer F.SilkS)
+    (effects (font (size 1.5 1.5) (thickness 0.18)))
+  )
+  (gr_text + (at 159.711331 52.797022 -191.3) (layer F.SilkS)
+    (effects (font (size 1.5 1.5) (thickness 0.18)))
+  )
+  (gr_text GND (at 162.43133 53.207022 -191.3) (layer F.SilkS)
+    (effects (font (size 1 1) (thickness 0.15)))
+  )
+  (gr_text S (at 157.231332 52.187021 -191.3) (layer F.SilkS)
+    (effects (font (size 1 1) (thickness 0.15)))
+  )
+  (gr_text S (at 137.767646 53.262718 -168.8) (layer F.SilkS)
+    (effects (font (size 1 1) (thickness 0.15)))
+  )
+  (gr_text + (at 140.292304 52.87723 -168.8) (layer F.SilkS)
+    (effects (font (size 1.5 1.5) (thickness 0.18)))
+  )
+  (gr_text GND (at 142.962155 52.215123 -168.8) (layer F.SilkS)
+    (effects (font (size 1 1) (thickness 0.15)))
+  )
+  (gr_text GND (at 125.426391 58.339901 -146.3) (layer F.SilkS)
+    (effects (font (size 1 1) (thickness 0.15)))
+  )
+  (gr_text + (at 123.213148 59.973316 -146.3) (layer F.SilkS)
+    (effects (font (size 1.5 1.5) (thickness 0.18)))
+  )
+  (gr_text S (at 121.028188 61.295606 -146.3) (layer F.SilkS)
+    (effects (font (size 1 1) (thickness 0.15)))
+  )
+  (gr_text S (at 108.364166 75.210708 -123.8) (layer F.SilkS)
+    (effects (font (size 1 1) (thickness 0.15)))
+  )
+  (gr_text GND (at 111.296477 70.796873 -123.8) (layer F.SilkS)
+    (effects (font (size 1 1) (thickness 0.15)))
+  )
+  (gr_text + (at 109.876788 73.152924 -123.8) (layer F.SilkS)
+    (effects (font (size 1.5 1.5) (thickness 0.18)))
+  )
+  (gr_text S (at 102.259176 93.417844 -101.3) (layer F.SilkS)
+    (effects (font (size 1 1) (thickness 0.15)))
+  )
+  (gr_text + (at 102.869176 90.937844 -101.3) (layer F.SilkS)
+    (effects (font (size 1.5 1.5) (thickness 0.18)))
+  )
+  (gr_text GND (at 103.279176 88.217845 -101.3) (layer F.SilkS)
+    (effects (font (size 1 1) (thickness 0.15)))
+  )
+  (gr_text S (at 103.324873 112.11153 -78.8) (layer F.SilkS)
+    (effects (font (size 1 1) (thickness 0.15)))
+  )
+  (gr_text + (at 102.939385 109.586872 -78.8) (layer F.SilkS)
+    (effects (font (size 1.5 1.5) (thickness 0.18)))
+  )
+  (gr_text GND (at 102.277277 106.91702 -78.8) (layer F.SilkS)
+    (effects (font (size 1 1) (thickness 0.15)))
+  )
+  (gr_text S (at 111.277761 128.700988 -56.3) (layer F.SilkS)
+    (effects (font (size 1 1) (thickness 0.15)))
+  )
+  (gr_text GND (at 108.322055 124.302784 -56.3) (layer F.SilkS)
+    (effects (font (size 1 1) (thickness 0.15)))
+  )
+  (gr_text + (at 109.955472 126.516028 -56.3) (layer F.SilkS)
+    (effects (font (size 1.5 1.5) (thickness 0.18)))
+  )
+  (gr_text GND (at 120.679028 138.352699 -33.8) (layer F.SilkS)
+    (effects (font (size 1 1) (thickness 0.15)))
+  )
+  (gr_text + (at 123.03508 139.772388 -33.8) (layer F.SilkS)
+    (effects (font (size 1.5 1.5) (thickness 0.18)))
+  )
+  (gr_text S (at 125.092864 141.28501 -33.8) (layer F.SilkS)
+    (effects (font (size 1 1) (thickness 0.15)))
+  )
+  (gr_text S (at 143.15 147.82 -11.3) (layer F.SilkS)
+    (effects (font (size 1 1) (thickness 0.15)))
+  )
+  (gr_text GND (at 137.95 146.8 -11.3) (layer F.SilkS)
+    (effects (font (size 1 1) (thickness 0.15)))
+  )
+  (gr_text + (at 140.67 147.21 -11.3) (layer F.SilkS)
+    (effects (font (size 1.5 1.5) (thickness 0.18)))
+  )
   (gr_text 10 (at 148.64 123.76) (layer F.SilkS)
