File: hw/motherboard/main/main.sch (KiCad schematic (older format))
At the start: 32 parts, among them J1 SWD holes, J10 stack[0..3], J11 stack[0..3], J12 stack[0..3], J13 GPIO, J2 Conn_ARM_JTAG_SWD_10, J4 STACK_GND, J9 stack[0..3], SW1 SW_Push, U1 STM32F303RETx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

Commit message: Board layouts before checking gerbers for alignment
Parts:
- removed J13: GPIO, Connector_PinSocket_2.54mm:PinSocket_1x08_P2.54mm_Vertical, symbol Connector:Conn_01x08_Female
- removed J4: STACK_GND, Connector_PinSocket_2.54mm:PinSocket_2x02_P2.54mm_Vertical, symbol Connector_Generic:Conn_02x02_Counter_Clockwise
- added J13: GPIO, Connector_PinHeader_2.54mm:PinHeader_2x04_P2.54mm_Vertical, symbol Connector_Generic:Conn_02x04_Counter_Clockwise
- added J4: STACK_GND, Connector_PinSocket_2.54mm:PinSocket_1x02_P2.54mm_Vertical, symbol Connector_Generic:Conn_01x02
Connections:
- net GND: now also J4.1 (Pin_1), J4.2 (Pin_2)
- net PA4: now also J13.1 (Pin_1)
- net PA5: now also J13.2 (Pin_2)
- net PA6: now also J13.3 (Pin_3)
- net PA7: now also J13.4 (Pin_4)
- net PB0: now also J13.8 (Pin_8)
- net PB12: now also J13.7 (Pin_7)
- net PC14: now also J13.6 (Pin_6)
- net PC15: now also J13.5 (Pin_5)
Changed lines of the file:
@@
 Text Notes 1700 3850 0    50   ~ 0
 Electromagnet control signals: m[0..15]\nPhoto gate sensor inputs: s[0..15]
-$Comp
-L power:GND #PWR095
-U 1 1 5F529F84
-P 2200 7000
-F 0 "#PWR095" H 2200 6750 50  0001 C CNN
-F 1 "GND" H 2205 6827 50  0000 C CNN
-F 2 "" H 2200 7000 50  0001 C CNN
-F 3 "" H 2200 7000 50  0001 C CNN
-	1    2200 7000
-	1    0    0    -1
-$EndComp
-Wire Wire Line
-	2200 7000 2200 6950
-$Comp
-L Connector_Generic:Conn_02x02_Counter_Clockwise J4
-U 1 1 5F5307C2
-P 2150 6750
-F 0 "J4" H 2200 6967 50  0000 C CNN
-F 1 "STACK_GND" H 2200 6876 50  0000 C CNN
-F 2 "Connector_PinSocket_2.54mm:PinSocket_2x02_P2.54mm_Vertical" H 2150 6750 50  0001 C CNN
-F 3 "~" H 2150 6750 50  0001 C CNN
-	1    2150 6750
-	1    0    0    -1
-$EndComp
-Wire Wire Line
-	1950 6750 1950 6850
-Wire Wire Line
-	1950 6950 2200 6950
-Connection ~ 1950 6850
-Wire Wire Line
-	1950 6850 1950 6950
-Wire Wire Line
-	2200 6950 2450 6950
-Wire Wire Line
-	2450 6950 2450 6850
-Connection ~ 2200 6950
-Connection ~ 2450 6850
-Wire Wire Line
-	2450 6850 2450 6750
 $Sheet
 S 750  3400 550  300
@@
 Wire Wire Line
 	6800 2800 6750 2800
-Text Label 8100 950  2    50   ~ 0
+Text Label 8250 950  2    50   ~ 0
 PA4
-Text Label 8100 1050 2    50   ~ 0
+Text Label 8250 1050 2    50   ~ 0
 PA5
-Text Label 8100 1150 2    50   ~ 0
+Text Label 8250 1150 2    50   ~ 0
 PA6
-Text Label 8100 1250 2    50   ~ 0
+Text Label 8250 1250 2    50   ~ 0
 PA7
 Text Label 6800 4100 0    50   ~ 0
@@
 Wire Wire Line
 	6800 4100 6750 4100
-Text Label 8100 1350 2    50   ~ 0
+Text Label 8750 950  0    50   ~ 0
 PB0
 Text Label 6800 5300 0    50   ~ 0
@@
 Wire Wire Line
 	6800 5300 6750 5300
-Text Label 8100 1450 2    50   ~ 0
+Text Label 8750 1050 0    50   ~ 0
 PB12
 Text Label 5300 5500 2    50   ~ 0
@@
 Wire Wire Line
 	5300 5600 5350 5600
-Text Label 8100 1550 2    50   ~ 0
+Text Label 8750 1150 0    50   ~ 0
 PC14
-Text Label 8100 1650 2    50   ~ 0
+Text Label 8750 1250 0    50   ~ 0
 PC15
 $Comp
-L Connector:Conn_01x08_Female J13
-U 1 1 5F5FAC84
-P 8300 1250
-F 0 "J13" H 8328 1226 50  0000 L CNN
-F 1 "GPIO" H 8328 1135 50  0000 L CNN
-F 2 "Connector_PinSocket_2.54mm:PinSocket_1x08_P2.54mm_Vertical" H 8300 1250 50  0001 C CNN
-F 3 "~" H 8300 1250 50  0001 C CNN
-	1    8300 1250
-	1    0    0    -1
-$EndComp
+L Connector_Generic:Conn_01x02 J4
+U 1 1 6017469B
+P 2200 6700
+F 0 "J4" H 2280 6692 50  0000 L CNN
+F 1 "STACK_GND" H 2280 6601 50  0000 L CNN
+F 2 "Connector_PinSocket_2.54mm:PinSocket_1x02_P2.54mm_Vertical" H 2200 6700 50  0001 C CNN
+F 3 "~" H 2200 6700 50  0001 C CNN
+	1    2200 6700
+	1    0    0    -1
+$EndComp
+Wire Wire Line
+	2000 6700 1950 6700
+Wire Wire Line
+	1950 6700 1950 6800
+Wire Wire Line
+	2000 6800 1950 6800
+Connection ~ 1950 6800
+Wire Wire Line
+	1950 6800 1950 6900
+$Comp
+L power:GND #PWR075
+U 1 1 601818C2
+P 1950 6900
+F 0 "#PWR075" H 1950 6650 50  0001 C CNN
+F 1 "GND" H 1955 6727 50  0000 C CNN
+F 2 "" H 1950 6900 50  0001 C CNN
+F 3 "" H 1950 6900 50  0001 C CNN
+	1    1950 6900
+	1    0    0    -1
+$EndComp
+$Comp
+L Connector_Generic:Conn_02x04_Counter_Clockwise J13
+U 1 1 601B22D7
+P 8450 1050
+F 0 "J13" H 8500 1367 50  0000 C CNN
+F 1 "GPIO" H 8500 1276 50  0000 C CNN
+F 2 "Connector_PinHeader_2.54mm:PinHeader_2x04_P2.54mm_Vertical" H 8450 1050 50  0001 C CNN
+F 3 "~" H 8450 1050 50  0001 C CNN
+	1    8450 1050
+	1    0    0    -1
+$EndComp
