File: hw/motherboard/main/power.sch (KiCad schematic (older format))
At the start: 12 parts, among them J6 5V power in, Q2 Q_PMOS_GSD, U3 LP5907MFX-3_3_NOPB, U4 TLV75533PDBV

Commit message: Finish laying out relelauta v2.0 PCB. Minor tweaks to motherboard.
Parts:
- removed J6: 5V power in, TerminalBlock:TerminalBlock_bornier-2_P5.08mm, symbol Connector:Conn_01x02_Male
- added J6: STACK_5V, Connector_PinSocket_2.54mm:PinSocket_2x02_P2.54mm_Vertical, symbol Connector_Generic:Conn_02x02_Counter_Clockwise
Connections:
- net labels added: 5V_in
- wire segments 43 -> 46
Other:
- note added: "Polarity protection"
- note removed: "TODO: verify pinout"
- moved on the sheet: C47, C48, C49, C50, D33, D34, Q2, R6, R7, U3, U4

Commit message: Board layouts before checking gerbers for alignment
Parts:
- removed J6: STACK_5V, Connector_PinSocket_2.54mm:PinSocket_2x02_P2.54mm_Vertical, symbol Connector_Generic:Conn_02x02_Counter_Clockwise
- added J6: STACK_5V, Connector_PinSocket_2.54mm:PinSocket_1x02_P2.54mm_Vertical, symbol Connector_Generic:Conn_01x02
Connections:
- net 5V_in: now also J6.1 (Pin_1), J6.2 (Pin_2)
Other:
- note added: "5V input from relelauta"
Changed lines of the file:
@@
 Wire Wire Line
 	3850 1850 3850 1950
+Text Notes 3550 1200 0    50   ~ 0
+Polarity protection
+Text Label 3150 1550 2    50   ~ 0
+5V_in
 $Comp
-L Connector_Generic:Conn_02x02_Counter_Clockwise J6
-U 1 1 60467FEA
-P 1750 1600
-F 0 "J6" H 1800 1300 50  0000 C CNN
-F 1 "STACK_5V" H 1800 1400 50  0000 C CNN
-F 2 "Connector_PinSocket_2.54mm:PinSocket_2x02_P2.54mm_Vertical" H 1750 1600 50  0001 C CNN
-F 3 "~" H 1750 1600 50  0001 C CNN
-	1    1750 1600
+L Connector_Generic:Conn_01x02 J6
+U 1 1 6019543D
+P 1600 1700
+F 0 "J6" H 1680 1692 50  0000 L CNN
+F 1 "STACK_5V" H 1680 1601 50  0000 L CNN
+F 2 "Connector_PinSocket_2.54mm:PinSocket_1x02_P2.54mm_Vertical" H 1600 1700 50  0001 C CNN
+F 3 "~" H 1600 1700 50  0001 C CNN
+	1    1600 1700
 	1    0    0    -1
 $EndComp
-Text Notes 3550 1200 0    50   ~ 0
-Polarity protection
+Text Label 1350 1600 0    50   ~ 0
+5V_in
 Wire Wire Line
-	2050 1700 2050 1600
+	1350 1600 1350 1700
 Wire Wire Line
-	2050 1500 1800 1500
+	1350 1800 1400 1800
 Wire Wire Line
-	1800 1500 1800 1450
-Connection ~ 2050 1600
+	1400 1700 1350 1700
+Connection ~ 1350 1700
 Wire Wire Line
-	2050 1600 2050 1500
-Wire Wire Line
-	1800 1500 1550 1500
-Wire Wire Line
-	1550 1500 1550 1600
-Connection ~ 1800 1500
-Connection ~ 1550 1600
-Wire Wire Line
-	1550 1600 1550 1700
-Text Label 1800 1450 0    50   ~ 0
-5V_in
-Text Label 3150 1550 2    50   ~ 0
-5V_in
+	1350 1700 1350 1800
+Text Notes 1100 1400 0    50   ~ 0
+5V input from relelauta
 $EndSCHEMATC
