File: hw/sensorilauta/sensorilauta.kicad_pcb (KiCad board)
At the start: 2 copper layers, 29.2 x 29.5 mm, 16 parts, among them J1 motherboard connector, Q1 Q_Photo_NPN, U1 MCP6001U

Commit message: Board layouts before checking gerbers for alignment
Parts:
- moved J1 0.28 mm to (96.0, 96.5)
Connections:
- J1 pad 1: /signal_out -> GND
- J1 pad 3: GND -> /signal_out
Routing:
- net /signal_out: track 30.3 -> 25.4 mm
