File: hw/sensorilauta/sensorilauta.sch (KiCad schematic (older format))
At the start: 16 parts, among them J1 motherboard connector, Q1 Q_Photo_NPN, U1 MCP6001U

Commit message: Board layouts before checking gerbers for alignment
Connections:
- net GND: now also J1.1 (Pin_1); no longer J1.3 (Pin_3)
- net signal_out: now also J1.3 (Pin_3); no longer J1.1 (Pin_1)
Changed lines of the file:
@@
 F 3 "~" H 7350 4000 50  0001 C CNN
 	1    7350 4000
-	1    0    0    -1
+	1    0    0    1
 $EndComp
 Text Label 7050 3900 2    50   ~ 0
